Commit message: Press buttons sequence working

File: initialize/models/block/model.urdf (robot description, URDF)
Before this commit: robot block, 1 links, 0 joints
Links:
- link block: geometry collision box size=0.03 0.03 0.03; visual box size=0.03 0.03 0.03

File: initialize/models/button/model.urdf (robot description, URDF)
Before this commit: robot button, 1 links, 0 joints
Links:
- link button: geometry collision box size=0.03 0.03 0.03; visual box size=0.03 0.03 0.03

Commit message: Added all servers and testClient

File: initialize/models/block/model.urdf (robot description, URDF)
Before this commit: robot block, 1 links, 0 joints
Links:
- link block: mass 1 -> 0.1
